File: IndicationPCB/IndicationPCB.kicad_pcb (KiCad board)
At the start: 2 copper layers, 14 x 32 mm, 6 parts, among them J1 Conn_01x03

Commit message: Draft
Routing:
- net +5V: track 27.4 -> 28.5 mm
Changed lines of the file:
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@@
+	)
+	(segment
+		(start 138.5 95)
+		(end 139 95.5)
+		(width 0.5)
+		(layer "F.Cu")
+		(net 2)
 	)
 	(segment
@@
 	)
 	(segment
+		(start 138.5 92.284652)
+		(end 138.5 95)
+		(width 0.5)
+		(layer "F.Cu")
+		(net 2)
+	)
+	(segment
 		(start 140.2 76.7)
 		(end 140.2 77.855008)
@@
 	)
 	(segment
+		(start 139.6959 91.088752)
+		(end 138.5 92.284652)
+		(width 0.5)
+		(layer "F.Cu")
+		(net 2)
+	)
+	(segment
 		(start 139.550001 86.677504)
 		(end 139 87.227505)
@@
 	)
 	(segment
-		(start 139.6959 91.088752)
-		(end 139 91.784652)
-		(width 0.5)
-		(layer "F.Cu")
-		(net 2)
-	)
-	(segment
 		(start 139.6959 82.266256)
 		(end 139.099 82.863156)
@@
 	)
 	(segment
-		(start 139 94.3)
-		(end 140.2 95.5)
-		(width 0.5)
-		(layer "F.Cu")
-		(net 2)
-	)
-	(segment
 		(start 139.6959 77.855008)
 		(end 139.099 78.451908)
@@
 	)
 	(segment
+		(start 139 95.5)
+		(end 140.2 95.5)
+		(width 0.5)
+		(layer "F.Cu")
+		(net 2)
+	)
+	(segment
 		(start 140.2 77.855008)
 		(end 139.6959 77.855008)
-		(width 0.5)
-		(layer "F.Cu")
-		(net 2)
-	)
-	(segment
-		(start 139 91.784652)
-		(end 139 94.3)
 		(width 0.5)
 		(layer "F.Cu")
@@
 	)
 	(segment
+		(start 144 87.677504)
+		(end 144.951 88.628504)
+		(width 0.2)
+		(layer "F.Cu")
+		(net 4)
+	)
+	(segment
 		(start 145.5 78.005007)
 		(end 145.5 76.5)
@@
 	)
 	(segment
+		(start 144.951 84.217256)
+		(end 144.951 87.376503)
+		(width 0.2)
+		(layer "F.Cu")
+		(net 4)
+	)
+	(segment
+		(start 144 92.088752)
+		(end 144.951 93.039752)
+		(width 0.2)
+		(layer "F.Cu")
+		(net 4)
+	)
+	(segment
+		(start 144 83.266256)
+		(end 144.951 84.217256)
+		(width 0.2)
+		(layer "F.Cu")
+		(net 4)
+	)
+	(segment
 		(start 144.649999 96.5)
 		(end 144 96.5)
@@
 	)
 	(segment
-		(start 144.951 84.217256)
-		(end 144.951 87.376503)
-		(width 0.2)
-		(layer "F.Cu")
-		(net 4)
-	)
-	(segment
-		(start 144 92.088752)
-		(end 144.951 93.039752)
+		(start 144.951 88.628504)
+		(end 144.951 91.787751)
+		(width 0.2)
+		(layer "F.Cu")
+		(net 4)
+	)
+	(segment
+		(start 144.951 91.787751)
+		(end 144.649999 92.088752)
+		(width 0.2)
+		(layer "F.Cu")
+		(net 4)
+	)
+	(segment
+		(start 144.951 87.376503)
+		(end 144.649999 87.677504)
+		(width 0.2)
+		(layer "F.Cu")
+		(net 4)
+	)
+	(segment
+		(start 144.951 96.198999)
+		(end 144.649999 96.5)
+		(width 0.2)
+		(layer "F.Cu")
+		(net 4)
+	)
+	(segment
+		(start 144.649999 78.855008)
+		(end 145.5 78.005007)
+		(width 0.2)
+		(layer "F.Cu")
+		(net 4)
+	)
+	(segment
+		(start 144.951 93.039752)
+		(end 144.951 96.198999)
+		(width 0.2)
+		(layer "F.Cu")
+		(net 4)
+	)
+	(segment
+		(start 144.649999 83.266256)
+		(end 144 83.266256)
+		(width 0.2)
+		(layer "F.Cu")
+		(net 4)
+	)
+	(segment
+		(start 144.649999 78.855008)
+		(end 144 78.855008)
+		(width 0.2)
+		(layer "F.Cu")
+		(net 4)
+	)
+	(segment
+		(start 144 78.855008)
+		(end 144.951 79.806008)
 		(width 0.2)
 		(layer "F.Cu")
@@
 		(start 144.649999 92.088752)
 		(end 144 92.088752)
-		(width 0.2)
-		(layer "F.Cu")
-		(net 4)
-	)
-	(segment
-		(start 144 83.266256)
-		(end 144.951 84.217256)
-		(width 0.2)
-		(layer "F.Cu")
-		(net 4)
-	)
-	(segment
-		(start 144.951 96.198999)
-		(end 144.649999 96.5)
-		(width 0.2)
-		(layer "F.Cu")
-		(net 4)
-	)
-	(segment
-		(start 144.951 87.376503)
-		(end 144.649999 87.677504)
-		(width 0.2)
-		(layer "F.Cu")
-		(net 4)
-	)
-	(segment
-		(start 144.951 93.039752)
-		(end 144.951 96.198999)
-		(width 0.2)
-		(layer "F.Cu")
-		(net 4)
-	)
-	(segment
-		(start 144.951 88.628504)
-		(end 144.951 91.787751)
-		(width 0.2)
-		(layer "F.Cu")
-		(net 4)
-	)
-	(segment
-		(start 144.649999 78.855008)
-		(end 145.5 78.005007)
-		(width 0.2)
-		(layer "F.Cu")
-		(net 4)
-	)
-	(segment
-		(start 144 87.677504)
-		(end 144.951 88.628504)
-		(width 0.2)
-		(layer "F.Cu")
-		(net 4)
-	)
-	(segment
-		(start 144.649999 83.266256)
-		(end 144 83.266256)
-		(width 0.2)
-		(layer "F.Cu")
-		(net 4)
-	)
-	(segment
-		(start 144.649999 78.855008)
-		(end 144 78.855008)
-		(width 0.2)
-		(layer "F.Cu")
-		(net 4)
-	)
-	(segment
-		(start 144.951 91.787751)
-		(end 144.649999 92.088752)
-		(width 0.2)
-		(layer "F.Cu")
-		(net 4)
-	)
-	(segment
-		(start 144 78.855008)
-		(end 144.951 79.806008)
 		(width 0.2)
 		(layer "F.Cu")
@@
 	)
 	(segment
-		(start 140.2 92.088752)
-		(end 140.2 92.388751)
+		(start 140.999 93.999)
+		(end 142.798999 93.999)
+		(width 0.2)
+		(layer "F.Cu")
+		(net 7)
+	)
+	(segment
+		(start 140.2 93.2)
+		(end 140.999 93.999)
 		(width 0.2)
 		(layer "F.Cu")
@@
 	)
 	(segment
-		(start 140.2 92.388751)
-		(end 141.810249 93.999)
-		(width 0.2)
-		(layer "F.Cu")
-		(net 7)
-	)
-	(segment
 		(start 144 95.200001)
 		(end 144 95.5)
@@
 	)
 	(segment
-		(start 141.810249 93.999)
-		(end 142.798999 93.999)
-		(width 0.2)
-		(layer "F.Cu")
+		(start 140.2 92.088752)
+		(end 140.2 93.2)
+		(width 0.2)
+		(layer "F.Cu")
