File: IndicationPCB.kicad_pcb (KiCad board)
At the start: 2 copper layers, 14.5 x 63 mm, 14 parts, among them J1 Conn_01x03

Commit message: bom
Parts:
- C4: value 1 uF -> 1uF
Changed lines of the file:
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@@
 			)
 		)
-		(property "Value" "1 uF"
+		(property "Value" "1uF"
 			(at 0 1.43 90)
 			(layer "F.Fab")
